File: KiCad/Sheets/06_RTC.kicad_sch (KiCad schematic)
At the start: 1 part, among them U9 DS3231+AT24C32

Commit message: Footprints are created and assigned
Parts:
- U9: footprint (none) -> Connector_PinSocket_2.54mm:PinSocket_1x06_P2.54mm_Vertical
Changed lines of the file:
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@@
 			)
 		)
-		(property "Footprint" ""
+		(property "Footprint" "Connector_PinSocket_2.54mm:PinSocket_1x06_P2.54mm_Vertical"
 			(at 151.13 101.6 0)
 			(hide yes)

Commit message: LEDs sheet added, schematic finished
Connections:
- net I2C_SCL: now also U9.3 (SCL); no longer U9.SCL
- net I2C_SDA: now also U9.4 (SDA); no longer U9.SDA
- net PWR_3V3_IN: now also U9.5 (VCC); no longer U9.VCC
- net PWR_GND: now also U9.6 (GND); no longer U9.GND
Changed lines of the file:
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@@
 			)
 		)
-		(pin "SQW"
+		(pin "5"
 		)
-		(pin "32K"
+		(pin "1"
 		)
-		(pin "GND"
+		(pin "2"
 		)
-		(pin "VCC"
+		(pin "3"
 		)
-		(pin "SDA"
+		(pin "6"
 		)
-		(pin "SCL"
+		(pin "4"
 		)
 		(instances
