File: KiCad/Sheets/09_MicroSD.kicad_sch (KiCad schematic)
At the start: 1 part, among them U11 MICROSD_SPI_3V3

Commit message: Footprints are created and assigned
Parts:
- U11: footprint (none) -> Connector_PinSocket_2.54mm:PinSocket_1x06_P2.54mm_Vertical
Changed lines of the file:
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@@
 			)
 		)
-		(property "Footprint" ""
+		(property "Footprint" "Connector_PinSocket_2.54mm:PinSocket_1x06_P2.54mm_Vertical"
 			(at 148.59 104.14 0)
 			(hide yes)

Commit message: LEDs sheet added, schematic finished
Connections:
- net MICROSD_CS: now also U11.2 (CS); no longer U11.CS
- net PWR_3V3_IN: now also U11.1 (3v3); no longer U11.3v3
- net PWR_GND: now also U11.6 (GND); no longer U11.GND
- net SPI_MISO: now also U11.5 (MISO); no longer U11.MISO
- net SPI_MOSI: now also U11.3 (MOSI); no longer U11.MOSI
- net SPI_SCK: now also U11.4 (CLK); no longer U11.CLK
Changed lines of the file:
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@@
 			)
 		)
-		(pin "3v3"
+		(pin "4"
 		)
-		(pin "MISO"
+		(pin "1"
 		)
-		(pin "GND"
+		(pin "6"
 		)
-		(pin "CLK"
+		(pin "3"
 		)
-		(pin "CS"
+		(pin "5"
 		)
-		(pin "MOSI"
+		(pin "2"
 		)
 		(instances
