File: KiCad/Sheets/07_Buzzer.kicad_sch (KiCad schematic)
At the start: 3 parts, among them Q1 S8050

Commit message: Footprints are created and assigned
Parts:
- added U19: CONN_JST_PH_2P, Connector_JST:JST_PH_B2B-PH-K_1x02_P2.00mm_Vertical, symbol HMS_Symbols:CONN_JST_PH_2P
- BZ1: footprint (none) -> Buzzer_Beeper:Buzzer_12x9.5RM7.6
- R3: footprint (none) -> Resistor_THT:R_Axial_DIN0207_L6.3mm_D2.5mm_P7.62mm_Horizontal
Connections:
- net PWR_5V_IN: now also U19.1
- net at BZ1.2 (-), Q1.3 (C): now also U19.2
Changed lines of the file:
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@@
 	(generator_version "10.0")
 	(paper "A4")
-	(text_box "JST connector"
-		(exclude_from_sim no)
-		(at 135.89 71.12 0)
-		(size 10.16 5.9929)
-		(margins 0.9525 0.9525 0.9525 0.9525)
-		(stroke
-			(width 0)
-			(type solid)
-		)
-		(fill
-			(type none)
-		)
-		(effects
-			(font
-				(size 1.27 1.27)
-			)
-			(justify top)
-		)
+	(junction
+		(at 139.7 72.39)
+		(diameter 0)
+		(color 255 0 0 1)
+	)
+	(junction
+		(at 142.24 72.39)
+		(diameter 0)
+		(color 0 0 0 1)
 	)
 	(wire
@@
 	(wire
 		(pts
-			(xy 139.7 52.07) (xy 139.7 91.44)
+			(xy 139.7 52.07) (xy 139.7 72.39)
 		)
 		(stroke
@@
 	(wire
 		(pts
+			(xy 142.24 72.39) (xy 142.24 91.44)
+		)
+		(stroke
+			(width 0.254)
+			(type default)
+			(color 0 0 0 1)
+		)
+	)
+	(wire
+		(pts
 			(xy 143.51 91.44) (xy 142.24 91.44)
 		)
@@
 	(wire
 		(pts
-			(xy 142.24 59.69) (xy 142.24 91.44)
+			(xy 139.7 72.39) (xy 139.7 91.44)
+		)
+		(stroke
+			(width 0.254)
+			(type default)
+			(color 255 0 0 1)
+		)
+	)
+	(wire
+		(pts
+			(xy 142.24 59.69) (xy 142.24 72.39)
 		)
 		(stroke
@@
 	)
 	(symbol
+		(lib_id "HMS_Symbols:CONN_JST_PH_2P")
+		(at 140.97 76.2 0)
+		(unit 1)
+		(body_style 1)
+		(exclude_from_sim no)
+		(in_bom yes)
+		(on_board yes)
+		(in_pos_files yes)
+		(dnp no)
+		(fields_autoplaced yes)
+		(property "Reference" "U19"
+			(at 146.05 74.9299 0)
+			(show_name no)
+			(do_not_autoplace no)
+			(effects
+				(font
+					(size 1.27 1.27)
+				)
+				(justify left)
+			)
+		)
+		(property "Value" "CONN_JST_PH_2P"
+			(at 146.05 77.4699 0)
+			(show_name no)
+			(do_not_autoplace no)
+			(effects
+				(font
+					(size 1.27 1.27)
+				)
+				(justify left)
+			)
+		)
+		(property "Footprint" "Connector_JST:JST_PH_B2B-PH-K_1x02_P2.00mm_Vertical"
+			(at 140.97 81.788 0)
+			(hide yes)
+			(show_name no)
+			(do_not_autoplace no)
+			(effects
+				(font
+					(size 1.27 1.27)
+				)
+			)
+		)
+		(property "Datasheet" ""
+			(at 140.97 76.2 0)
+			(hide yes)
+			(show_name no)
+			(do_not_autoplace no)
+			(effects
+				(font
+					(size 1.27 1.27)
+				)
+			)
+		)
+		(property "Description" ""
+			(at 140.97 76.2 0)
+			(hide yes)
+			(show_name no)
+			(do_not_autoplace no)
+			(effects
+				(font
+					(size 1.27 1.27)
+				)
+			)
+		)
+		(pin "2"
+		)
+		(pin "1"
+		)
+		(instances
+			(project "HMS_Master"
+				(path "/cab65a7d-0a7e-481c-9f85-25eca3c1fa1e/a2e28c65-40dc-4ab8-b49b-8c9d90f9a40b"
+					(reference "U19")
+					(unit 1)
+				)
+			)
+		)
+	)
+	(symbol
 		(lib_id "Device:R")
 		(at 147.32 45.72 0)
@@
 			)
 		)
-		(property "Footprint" ""
+		(property "Footprint" "Resistor_THT:R_Axial_DIN0207_L6.3mm_D2.5mm_P7.62mm_Horizontal"
 			(at 145.542 45.72 90)
 			(hide yes)
@@
 			)
 		)
-		(property "Footprint" ""
+		(property "Footprint" "Buzzer_Beeper:Buzzer_12x9.5RM7.6"
 			(at 138.43 95.885 90)
 			(hide yes)

Commit message: LEDs sheet added, schematic finished
Parts:
- U19: value CONN_JST_PH_2P -> BUZZER_SOCKET
Changed lines of the file:
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@@
 			)
 		)
-		(property "Value" "CONN_JST_PH_2P"
+		(property "Value" "BUZZER_SOCKET"
 			(at 146.05 77.4699 0)
 			(show_name no)
@@
 		(exclude_from_sim no)
 		(in_bom yes)
-		(on_board yes)
+		(on_board no)
 		(in_pos_files yes)
 		(dnp no)

Commit message: Finished PCB
Parts:
- Q1: footprint Package_TO_SOT_THT:TO-92_Inline -> Package_TO_SOT_THT:TO-92_Inline_Wide
- U19: footprint Connector_JST:JST_PH_B2B-PH-K_1x02_P2.00mm_Vertical -> Connector_JST:JST_XH_B2B-XH-A_1x02_P2.50mm_Vertical
Changed lines of the file:
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@@
 			)
 		)
-		(property "Footprint" "Package_TO_SOT_THT:TO-92_Inline"
+		(property "Footprint" "Package_TO_SOT_THT:TO-92_Inline_Wide"
 			(at 149.225 62.23 0)
 			(hide yes)
@@
 			)
 		)
-		(property "Footprint" "Connector_JST:JST_PH_B2B-PH-K_1x02_P2.00mm_Vertical"
+		(property "Footprint" "Connector_JST:JST_XH_B2B-XH-A_1x02_P2.50mm_Vertical"
 			(at 140.97 81.788 0)
 			(hide yes)
