File: KiCad/Sheets/08_Boiler_Room_Sensor.kicad_sch (KiCad schematic)
At the start: 1 part, among them U10 DHT11

Commit message: Footprints are created and assigned
Parts:
- added U20: CONN_JST_PH_3P, Connector_JST:JST_PH_B3B-PH-K_1x03_P2.00mm_Vertical, symbol HMS_Symbols:CONN_JST_PH_3P
- U10: footprint Sensor:Aosong_DHT11_5.5x12.0_P2.54mm -> Connector_PinSocket_2.54mm:PinSocket_1x03_P2.54mm_Vertical
Connections:
- net BOILER_ROOM_TEMPERATURE: now also U20.2
- net PWR_3V3_IN: now also U20.1
- net PWR_GND: now also U20.3
Changed lines of the file:
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@@
 	(generator_version "10.0")
 	(paper "A4")
-	(text_box "JST connector"
-		(exclude_from_sim no)
-		(at 130.81 77.47 0)
-		(size 10.16 5.9929)
-		(margins 0.9525 0.9525 0.9525 0.9525)
-		(stroke
-			(width 0)
-			(type solid)
-		)
-		(fill
-			(type none)
-		)
-		(effects
-			(font
-				(size 1.27 1.27)
-			)
-			(justify top)
-		)
-	)
-	(wire
-		(pts
-			(xy 133.35 69.85) (xy 133.35 91.44)
+	(junction
+		(at 133.35 74.93)
+		(diameter 0)
+		(color 0 0 0 0)
+	)
+	(junction
+		(at 135.89 74.93)
+		(diameter 0)
+		(color 0 0 0 0)
+	)
+	(junction
+		(at 138.43 74.93)
+		(diameter 0)
+		(color 0 0 0 0)
+	)
+	(wire
+		(pts
+			(xy 133.35 69.85) (xy 133.35 74.93)
 		)
 		(stroke
@@
 	(wire
 		(pts
-			(xy 135.89 69.85) (xy 135.89 95.25)
+			(xy 135.89 69.85) (xy 135.89 74.93)
 		)
 		(stroke
@@
 	(wire
 		(pts
-			(xy 138.43 69.85) (xy 138.43 91.44)
-		)
-		(stroke
-			(width 0.254)
-			(type default)
-			(color 0 0 0 1)
+			(xy 138.43 74.93) (xy 138.43 91.44)
+		)
+		(stroke
+			(width 0.254)
+			(type default)
+			(color 0 0 0 1)
+		)
+	)
+	(wire
+		(pts
+			(xy 138.43 69.85) (xy 138.43 74.93)
+		)
+		(stroke
+			(width 0.254)
+			(type default)
+			(color 0 0 0 1)
+		)
+	)
+	(wire
+		(pts
+			(xy 135.89 74.93) (xy 135.89 95.25)
+		)
+		(stroke
+			(width 0.254)
+			(type default)
+			(color 194 194 194 1)
+		)
+	)
+	(wire
+		(pts
+			(xy 133.35 74.93) (xy 133.35 91.44)
+		)
+		(stroke
+			(width 0.254)
+			(type default)
+			(color 255 0 0 1)
 		)
 	)
@@
 			)
 			(justify left)
+		)
+	)
+	(symbol
+		(lib_id "HMS_Symbols:CONN_JST_PH_3P")
+		(at 135.89 78.74 0)
+		(unit 1)
+		(body_style 1)
+		(exclude_from_sim no)
+		(in_bom yes)
+		(on_board yes)
+		(in_pos_files yes)
+		(dnp no)
+		(fields_autoplaced yes)
+		(property "Reference" "U20"
+			(at 142.24 77.4699 0)
+			(show_name no)
+			(do_not_autoplace no)
+			(effects
+				(font
+					(size 1.27 1.27)
+				)
+				(justify left)
+			)
+		)
+		(property "Value" "CONN_JST_PH_3P"
+			(at 142.24 80.0099 0)
+			(show_name no)
+			(do_not_autoplace no)
+			(effects
+				(font
+					(size 1.27 1.27)
+				)
+				(justify left)
+			)
+		)
+		(property "Footprint" "Connector_JST:JST_PH_B3B-PH-K_1x03_P2.00mm_Vertical"
+			(at 135.89 85.852 0)
+			(hide yes)
+			(show_name no)
+			(do_not_autoplace no)
+			(effects
+				(font
+					(size 1.27 1.27)
+				)
+			)
+		)
+		(property "Datasheet" ""
+			(at 135.89 78.74 0)
+			(hide yes)
+			(show_name no)
+			(do_not_autoplace no)
+			(effects
+				(font
+					(size 1.27 1.27)
+				)
+			)
+		)
+		(property "Description" ""
+			(at 135.89 78.74 0)
+			(hide yes)
+			(show_name no)
+			(do_not_autoplace no)
+			(effects
+				(font
+					(size 1.27 1.27)
+				)
+			)
+		)
+		(pin "2"
+		)
+		(pin "1"
+		)
+		(pin "3"
+		)
+		(instances
+			(project "HMS_Master"
+				(path "/cab65a7d-0a7e-481c-9f85-25eca3c1fa1e/90b74869-0313-4dc3-8b6e-6d6576565e56"
+					(reference "U20")
+					(unit 1)
+				)
+			)
 		)
 	)
@@
 			)
 		)
-		(property "Footprint" "Sensor:Aosong_DHT11_5.5x12.0_P2.54mm"
+		(property "Footprint" "Connector_PinSocket_2.54mm:PinSocket_1x03_P2.54mm_Vertical"
 			(at 146.05 102.87 0)
 			(hide yes)

Commit message: LEDs sheet added, schematic finished
Parts:
- U10: footprint Connector_PinSocket_2.54mm:PinSocket_1x03_P2.54mm_Vertical -> Sensor:Aosong_DHT11_5.5x12.0_P2.54mm
- U20: value CONN_JST_PH_3P -> BOILER_ROOM_SENSOR_SOCKET
Changed lines of the file:
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@@
 		(at 133.35 74.93)
 		(diameter 0)
-		(color 0 0 0 0)
+		(color 255 0 0 1)
 	)
 	(junction
 		(at 135.89 74.93)
 		(diameter 0)
-		(color 0 0 0 0)
+		(color 194 194 194 1)
 	)
 	(junction
 		(at 138.43 74.93)
 		(diameter 0)
-		(color 0 0 0 0)
+		(color 0 0 0 1)
 	)
 	(wire
@@
 			)
 		)
-		(property "Value" "CONN_JST_PH_3P"
+		(property "Value" "BOILER_ROOM_SENSOR_SOCKET"
 			(at 142.24 80.0099 0)
 			(show_name no)
@@
 		(exclude_from_sim no)
 		(in_bom yes)
-		(on_board yes)
+		(on_board no)
 		(in_pos_files yes)
 		(dnp no)
@@
 			)
 		)
-		(property "Footprint" "Connector_PinSocket_2.54mm:PinSocket_1x03_P2.54mm_Vertical"
+		(property "Footprint" "Sensor:Aosong_DHT11_5.5x12.0_P2.54mm"
 			(at 146.05 102.87 0)
 			(hide yes)

Commit message: Finished PCB
Parts:
- U20: footprint Connector_JST:JST_PH_B3B-PH-K_1x03_P2.00mm_Vertical -> Connector_JST:JST_XH_B3B-XH-A_1x03_P2.50mm_Vertical
Changed lines of the file:
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@@
 			)
 		)
-		(property "Footprint" "Connector_JST:JST_PH_B3B-PH-K_1x03_P2.00mm_Vertical"
+		(property "Footprint" "Connector_JST:JST_XH_B3B-XH-A_1x03_P2.50mm_Vertical"
 			(at 135.89 85.852 0)
 			(hide yes)
