File: KiCad/Sheets/11_LEDs.kicad_sch (KiCad schematic)
At the start: 17 parts, among them U27 SERVO16-1A-SLD, U30 LED_GAS_SOCKET, U31 LED_WOOD_SOCKET, U32 LED_STATUS_SOCKET

Commit message: Finished PCB
Parts:
- U30, U31, U32: footprint Connector_JST:JST_PH_B4B-PH-K_1x04_P2.00mm_Vertical -> Connector_JST:JST_XH_B4B-XH-A_1x04_P2.50mm_Vertical
Connections:
- no-connect marks 10 -> 8
Changed lines of the file:
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@@
-	)
-	(no_connect
-		(at 156.21 140.97)
-	)
-	(no_connect
-		(at 156.21 137.16)
 	)
 	(no_connect
@@
 		(pin "20"
 		)
-		(pin "23"
-		)
 		(pin "17"
 		)
@@
 		)
 		(pin "18"
-		)
-		(pin "24"
 		)
 		(pin "21"
@@
 			)
 		)
-		(property "Footprint" "Connector_JST:JST_PH_B4B-PH-K_1x04_P2.00mm_Vertical"
+		(property "Footprint" "Connector_JST:JST_XH_B4B-XH-A_1x04_P2.50mm_Vertical"
 			(at 205.994 91.44 0)
 			(hide yes)
@@
 			)
 		)
-		(property "Footprint" "Connector_JST:JST_PH_B4B-PH-K_1x04_P2.00mm_Vertical"
+		(property "Footprint" "Connector_JST:JST_XH_B4B-XH-A_1x04_P2.50mm_Vertical"
 			(at 205.994 74.93 0)
 			(hide yes)
@@
 			)
 		)
-		(property "Footprint" "Connector_JST:JST_PH_B4B-PH-K_1x04_P2.00mm_Vertical"
+		(property "Footprint" "Connector_JST:JST_XH_B4B-XH-A_1x04_P2.50mm_Vertical"
 			(at 205.994 107.95 0)
 			(hide yes)
