File: KiCad/HMS_Master/HMS_Master.kicad_sch (KiCad schematic)
At the start: 0 parts

Commit message: Refactor KiCad Master directory structure
Other:
- sheet 01_ESP32: file ../Sheets/01_ESP32.kicad_sch -> Sheets/01_ESP32.kicad_sch
- sheet 02_Power_Supply: file ../Sheets/02_Power_Supply.kicad_sch -> Sheets/02_Power_Supply.kicad_sch
- sheet 03_Display: file ../Sheets/03_Display.kicad_sch -> Sheets/03_Display.kicad_sch
- sheet 04_Chimney_Temperature: file ../Sheets/04_Chimney_Temperature.kicad_sch -> Sheets/04_Chimney_Temperature.kicad_sch
- sheet 05_Temperature_Sensors: file ../Sheets/05_Temperature_Sensors.kicad_sch -> Sheets/05_Temperature_Sensors.kicad_sch
- sheet 06_RTC: file ../Sheets/06_RTC.kicad_sch -> Sheets/06_RTC.kicad_sch
- sheet 07_Buzzer: file ../Sheets/07_Buzzer.kicad_sch -> Sheets/07_Buzzer.kicad_sch
- sheet 08_Boiler_Room_Sensor: file ../Sheets/08_Boiler_Room_Sensor.kicad_sch -> Sheets/08_Boiler_Room_Sensor.kicad_sch
- sheet 09_MicroSD: file ../Sheets/09_MicroSD.kicad_sch -> Sheets/09_MicroSD.kicad_sch
- sheet 10_Voltage_Detectors: file ../Sheets/10_Voltage_Detectors.kicad_sch -> Sheets/10_Voltage_Detectors.kicad_sch
- sheet 11_LEDs: file ../Sheets/11_LEDs.kicad_sch -> Sheets/11_LEDs.kicad_sch
Changed lines of the file:
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@@
 			)
 		)
-		(property "Sheetfile" "../Sheets/03_Display.kicad_sch"
+		(property "Sheetfile" "Sheets/03_Display.kicad_sch"
 			(at 101.6 76.7846 0)
 			(show_name no)
@@
 			)
 		)
-		(property "Sheetfile" "../Sheets/01_ESP32.kicad_sch"
+		(property "Sheetfile" "Sheets/01_ESP32.kicad_sch"
 			(at 44.45 243.1546 0)
 			(show_name no)
@@
 			)
 		)
-		(property "Sheetfile" "../Sheets/08_Boiler_Room_Sensor.kicad_sch"
+		(property "Sheetfile" "Sheets/08_Boiler_Room_Sensor.kicad_sch"
 			(at 101.6 179.6546 0)
 			(show_name no)
@@
 			)
 		)
-		(property "Sheetfile" "../Sheets/06_RTC.kicad_sch"
+		(property "Sheetfile" "Sheets/06_RTC.kicad_sch"
 			(at 101.6 140.2846 0)
 			(show_name no)
@@
 			)
 		)
-		(property "Sheetfile" "../Sheets/07_Buzzer.kicad_sch"
+		(property "Sheetfile" "Sheets/07_Buzzer.kicad_sch"
 			(at 101.6 158.0646 0)
 			(show_name no)
@@
 			)
 		)
-		(property "Sheetfile" "../Sheets/09_MicroSD.kicad_sch"
+		(property "Sheetfile" "Sheets/09_MicroSD.kicad_sch"
 			(at 101.6 207.5946 0)
 			(show_name no)
@@
 			)
 		)
-		(property "Sheetfile" "../Sheets/02_Power_Supply.kicad_sch"
+		(property "Sheetfile" "Sheets/02_Power_Supply.kicad_sch"
 			(at 44.45 29.7946 0)
 			(show_name no)
@@
 			)
 		)
-		(property "Sheetfile" "../Sheets/10_Voltage_Detectors.kicad_sch"
+		(property "Sheetfile" "Sheets/10_Voltage_Detectors.kicad_sch"
 			(at 101.6 225.3746 0)
 			(show_name no)
@@
 			)
 		)
-		(property "Sheetfile" "../Sheets/05_Temperature_Sensors.kicad_sch"
+		(property "Sheetfile" "Sheets/05_Temperature_Sensors.kicad_sch"
 			(at 101.6 122.5046 0)
 			(show_name no)
@@
 			)
 		)
-		(property "Sheetfile" "../Sheets/04_Chimney_Temperature.kicad_sch"
+		(property "Sheetfile" "Sheets/04_Chimney_Temperature.kicad_sch"
 			(at 101.6 100.9146 0)
 			(show_name no)
@@
 			)
 		)
-		(property "Sheetfile" "../Sheets/11_LEDs.kicad_sch"
+		(property "Sheetfile" "Sheets/11_LEDs.kicad_sch"
 			(at 101.6 243.1546 0)
 			(show_name no)
