File: KiCad/HMS_Master/Sheets/01_ESP32.kicad_sch (KiCad schematic)
At the start: 1 part, among them U1 ESP32-DEVKITC-32UE

Commit message: Refactor KiCad Master directory structure
Other:
- moved on the sheet: U1
Changed lines of the file:
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@@
 	)
 	(junction
-		(at 158.75 60.96)
+		(at 158.75 83.82)
 		(diameter 0)
 		(color 0 0 0 1)
 	)
 	(junction
-		(at 121.92 87.63)
+		(at 121.92 110.49)
 		(diameter 0)
 		(color 0 0 0 1)
 	)
 	(no_connect
-		(at 121.92 45.72)
-	)
-	(no_connect
-		(at 177.8 49.53)
-	)
-	(no_connect
-		(at 177.8 53.34)
-	)
-	(no_connect
-		(at 121.92 83.82)
-	)
-	(no_connect
-		(at 121.92 99.06)
-	)
-	(no_connect
-		(at 121.92 49.53)
-	)
-	(no_connect
-		(at 121.92 41.91)
-	)
-	(no_connect
-		(at 121.92 57.15)
-	)
-	(no_connect
-		(at 177.8 91.44)
-	)
-	(no_connect
-		(at 121.92 102.87)
-	)
-	(no_connect
-		(at 177.8 87.63)
-	)
-	(no_connect
-		(at 177.8 102.87)
-	)
-	(no_connect
-		(at 121.92 53.34)
-	)
-	(no_connect
-		(at 177.8 99.06)
-	)
-	(no_connect
-		(at 121.92 95.25)
-	)
-	(no_connect
-		(at 177.8 106.68)
-	)
-	(no_connect
-		(at 177.8 95.25)
-	)
-	(wire
-		(pts
-			(xy 158.75 38.1) (xy 158.75 60.96)
+		(at 121.92 68.58)
+	)
+	(no_connect
+		(at 177.8 72.39)
+	)
+	(no_connect
+		(at 177.8 76.2)
+	)
+	(no_connect
+		(at 121.92 106.68)
+	)
+	(no_connect
+		(at 121.92 121.92)
+	)
+	(no_connect
+		(at 121.92 72.39)
+	)
+	(no_connect
+		(at 121.92 64.77)
+	)
+	(no_connect
+		(at 121.92 80.01)
+	)
+	(no_connect
+		(at 177.8 114.3)
+	)
+	(no_connect
+		(at 121.92 125.73)
+	)
+	(no_connect
+		(at 177.8 110.49)
+	)
+	(no_connect
+		(at 177.8 125.73)
+	)
+	(no_connect
+		(at 121.92 76.2)
+	)
+	(no_connect
+		(at 177.8 121.92)
+	)
+	(no_connect
+		(at 121.92 118.11)
+	)
+	(no_connect
+		(at 177.8 129.54)
+	)
+	(no_connect
+		(at 177.8 118.11)
+	)
+	(wire
+		(pts
+			(xy 158.75 60.96) (xy 158.75 83.82)
 		)
 		(stroke
@@
 	(wire
 		(pts
-			(xy 158.75 60.96) (xy 158.75 87.63)
+			(xy 158.75 83.82) (xy 158.75 110.49)
 		)
 		(stroke
@@
 	(wire
 		(pts
-			(xy 158.75 60.96) (xy 177.8 60.96)
+			(xy 158.75 83.82) (xy 177.8 83.82)
 		)
 		(stroke
@@
 	(wire
 		(pts
-			(xy 177.8 38.1) (xy 158.75 38.1)
+			(xy 177.8 60.96) (xy 158.75 60.96)
 		)
 		(stroke
@@
 	(wire
 		(pts
-			(xy 113.03 106.68) (xy 121.92 106.68)
+			(xy 113.03 129.54) (xy 121.92 129.54)
 		)
 		(stroke
@@
 	(wire
 		(pts
-			(xy 111.76 87.63) (xy 121.92 87.63)
+			(xy 111.76 110.49) (xy 121.92 110.49)
 		)
 		(stroke
@@
 	(wire
 		(pts
-			(xy 121.92 87.63) (xy 158.75 87.63)
+			(xy 121.92 110.49) (xy 158.75 110.49)
 		)
 		(stroke
@@
 	(hierarchical_label "DISPLAY_RESET"
 		(shape output)
-		(at 177.8 80.01 0)
+		(at 177.8 102.87 0)
 		(effects
 			(font
@@
 	(hierarchical_label "CHIMNEY_TEMPERATURE_CS"
 		(shape input)
-		(at 121.92 80.01 180)
+		(at 121.92 102.87 180)
 		(effects
 			(font
@@
 	(hierarchical_label "SPI_SCK"
 		(shape output)
-		(at 177.8 68.58 0)
+		(at 177.8 91.44 0)
 		(effects
 			(font
@@
 	(hierarchical_label "DISPLAY1_CS"
 		(shape output)
-		(at 177.8 72.39 0)
+		(at 177.8 95.25 0)
 		(effects
 			(font
@@
 	(hierarchical_label "DISPLAY2_CS"
 		(shape output)
-		(at 177.8 83.82 0)
+		(at 177.8 106.68 0)
 		(effects
 			(font
@@
 	(hierarchical_label "I2C_SDA"
 		(shape bidirectional)
-		(at 177.8 57.15 0)
+		(at 177.8 80.01 0)
 		(effects
 			(font
@@
 	(hierarchical_label "BUZZER"
 		(shape output)
-		(at 121.92 68.58 180)
+		(at 121.92 91.44 180)
 		(effects
 			(font
@@
 	(hierarchical_label "PWR_3V3_OUT"
 		(shape output)
-		(at 121.92 38.1 180)
+		(at 121.92 60.96 180)
 		(effects
 			(font
@@
 	(hierarchical_label "TEMPERATURE_SENSOR_BUS"
 		(shape input)
-		(at 121.92 76.2 180)
+		(at 121.92 99.06 180)
 		(effects
 			(font
@@
 	(hierarchical_label "PWR_5V_IN"
 		(shape input)
-		(at 113.03 106.68 180)
+		(at 113.03 129.54 180)
 		(effects
 			(font
@@
 	(hierarchical_label "BOILER_ROOM_TEMPERATURE"
 		(shape input)
-		(at 121.92 72.39 180)
+		(at 121.92 95.25 180)
 		(effects
 			(font
@@
 	(hierarchical_label "PWR_GND"
 		(shape input)
-		(at 111.76 87.63 180)
+		(at 111.76 110.49 180)
 		(effects
 			(font
@@
 	(hierarchical_label "SPI_MISO"
 		(shape input)
+		(at 177.8 87.63 0)
+		(effects
+			(font
+				(size 1.27 1.27)
+			)
+			(justify left)
+		)
+	)
+	(hierarchical_label "DISPLAY_DC"
+		(shape output)
+		(at 177.8 99.06 0)
+		(effects
+			(font
+				(size 1.27 1.27)
+			)
+			(justify left)
+		)
+	)
+	(hierarchical_label "SPI_MOSI"
+		(shape output)
 		(at 177.8 64.77 0)
 		(effects
@@
 		)
 	)
-	(hierarchical_label "DISPLAY_DC"
-		(shape output)
-		(at 177.8 76.2 0)
-		(effects
-			(font
-				(size 1.27 1.27)
-			)
-			(justify left)
-		)
-	)
-	(hierarchical_label "SPI_MOSI"
-		(shape output)
-		(at 177.8 41.91 0)
-		(effects
-			(font
-				(size 1.27 1.27)
-			)
-			(justify left)
-		)
-	)
 	(hierarchical_label "MICROSD_CS"
 		(shape output)
-		(at 121.92 91.44 180)
+		(at 121.92 114.3 180)
 		(effects
 			(font
@@
 	(hierarchical_label "WOOD_AC_PRESENT"
 		(shape input)
-		(at 121.92 64.77 180)
+		(at 121.92 87.63 180)
 		(effects
 			(font
@@
 	(hierarchical_label "GAS_AC_PRESENT"
 		(shape input)
-		(at 121.92 60.96 180)
+		(at 121.92 83.82 180)
 		(effects
 			(font
@@
 	(hierarchical_label "I2C_SCL"
 		(shape output)
-		(at 177.8 45.72 0)
+		(at 177.8 68.58 0)
 		(effects
 			(font
@@
 	(symbol
 		(lib_id "HMS_Symbols:ESP32_DEVKITC_32UE")
-		(at 134.62 34.29 0)
+		(at 134.62 57.15 0)
 		(unit 1)
 		(body_style 1)
@@
 		(fields_autoplaced yes)
 		(property "Reference" "U1"
-			(at 149.86 31.75 0)
+			(at 149.86 54.61 0)
 			(show_name no)
 			(do_not_autoplace no)
@@
 		)
 		(property "Value" "ESP32-DEVKITC-32UE"
-			(at 149.86 34.29 0)
+			(at 149.86 57.15 0)
 			(show_name no)
 			(do_not_autoplace no)
@@
 		)
 		(property "Footprint" "HMS_Footprints:ESP32_DEVKITC_32UE"
-			(at 134.62 34.29 0)
+			(at 134.62 57.15 0)
 			(hide yes)
 			(show_name no)
@@
 		)
 		(property "Datasheet" "https://docs.espressif.com/projects/esp-dev-kits/en/latest/esp32/esp32-devkitc/user_guide.html#id11"
-			(at 149.606 30.226 0)
+			(at 149.606 53.086 0)
 			(hide yes)
 			(show_name no)
@@
 		)
 		(property "Description" "ESP32-DEVKITC-32UE development board based on ESP32-WROOM-32UE."
-			(at 151.638 27.686 0)
+			(at 151.638 50.546 0)
 			(hide yes)
 			(show_name no)
@@
 		)
 		(property "Description2" "Reserved pins: SD0, SD1, SD2, SD3, CMD and CLK are connected to the internal flash and must not be used."
-			(at 149.606 32.258 0)
+			(at 149.606 55.118 0)
 			(hide yes)
 			(show_name no)
@@
 		)
 		(property "Description3" "Only one GND pin needs to be connected in the schematic."
-			(at 134.62 34.29 0)
+			(at 134.62 57.15 0)
 			(hide yes)
 			(show_name no)
@@
 		)
 		(property "Description4" "All GND pins of the module must be connected on the PCB."
-			(at 134.62 34.29 0)
+			(at 134.62 57.15 0)
 			(hide yes)
 			(show_name no)
@@
 		)
 		(property "Descriton2" "Reserved pins: SD0, SD1, SD2, SD3, CMD and CLK are connected to the internal flash and must not be used."
-			(at 149.606 32.258 0)
+			(at 149.606 55.118 0)
 			(hide yes)
 			(show_name no)
@@
 		)
 	)
-	(sheet_instances
-		(path "/"
-			(page "1")
-		)
-	)
