File: KiCad/HMS_Master/Sheets/07_Buzzer.kicad_sch (KiCad schematic)
At the start: 4 parts, among them U26 USB_Micro-B_Socket

Commit message: Refactor KiCad Master directory structure
Parts:
- removed C1470µF/10V1: 470µF 10V, Capacitor_THT:CP_Radial_D8.0mm_P3.50mm, symbol Device:C_Polarized
- removed C2100nF/50V1: 100nF 50V, Capacitor_THT:C_Disc_D3.8mm_W2.6mm_P2.50mm, symbol Device:C
- removed F1: T1A Fuse, Fuse:Fuseholder_Cylinder-5x20mm_Schurter_0031_8201_Horizontal_Open, symbol Device:Fuse
- removed U26: USB_Micro-B_Socket, Connector_JST:JST_XH_B2B-XH-A_1x02_P2.50mm_Vertical, symbol HMS_Symbols:CONN_JST_PH_2P
- added BZ1: Buzzer, Buzzer_Beeper:Buzzer_12x9.5RM7.6, symbol Device:Buzzer
- added Q1: S8050, Package_TO_SOT_THT:TO-92_Inline_Wide, symbol Transistor_BJT:S8050
- added R3: 1kΩ, Resistor_THT:R_Axial_DIN0207_L6.3mm_D2.5mm_P7.62mm_Horizontal, symbol Device:R
- added U19: BUZZER_SOCKET, Connector_JST:JST_XH_B2B-XH-A_1x02_P2.50mm_Vertical, symbol HMS_Symbols:CONN_JST_PH_2P
Connections:
- net PWR_GND: now also Q1.1 (E)
- new net: Q1.2 (B), R3.2
- new net: BZ1.2 (-), Q1.3 (C), U19.2
- new net BUZZER: R3.1
- new net PWR_5V_IN: BZ1.1 (+), U19.1
Other:
- note removed: "POWER SUPPLY"
- title: HMS-Master -> (none)
