File: KiCad/HMS_Display/HMS_Display.kicad_sch (KiCad schematic)
At the start: 0 parts

Commit message: HMS_Diaply Kicad schematics and PCB
Other:
- added sheet 01_ESP32 (Sheets/01_ESP32.kicad_sch)
- added sheet 02_Power_Supply (Sheets/02_Power_Supply.kicad_sch)
- added sheet 03_Display (Sheets/03_Display.kicad_sch)
- added sheet 04_Temperature_Sensor (Sheets/04_Temperature_Sensor.kicad_sch)
- added sheet 05_RTC (Sheets/05_RTC.kicad_sch)
- added sheet 06_Buzzer (Sheets/06_Buzzer.kicad_sch)
- added sheet 07_LEDs (Sheets/07_LEDs.kicad_sch)
- added sheet 08_Photoresistor (Sheets\08_Photoresistor.kicad_sch)
- title: (none) -> HMS-Master
