File: KiCad/HMS_Display/Sheets/01_ESP32.kicad_sch (KiCad schematic)
At the start: 1 part, among them U1 ESP32-DEVKITC-32UE

Commit message: HMS_Diaply Kicad schematics and PCB
Parts:
- U1: footprint HMS_Footprints:ESP32_DEVKITC_32UE -> HMS:ESP32_DEVKITC_32UE
Connections:
- net DISPLAY2_CS is gone; now on net DISPLAY_RESET: U1.32 (GPIO4)
- net DISPLAY_DC: now also U1.31 (GPIO16); no longer U1.30 (GPIO17)
- net DISPLAY_RESET: no longer U1.31 (GPIO16)
- net T_IRQ: now reaches U1.5 (GPIO34)
- net PHOTORESISTOR: now reaches U1.6 (GPIO35)
- net BOILER_ROOM_TEMPERATURE renamed LED_B
- net BUZZER renamed LED_G
- net CHIMNEY_TEMPERATURE_CS renamed BUZZER_1
- net DISPLAY1_CS: no longer names the net of U1.29 (GPIO5)
- net GAS_AC_PRESENT renamed DISPLAY_LED
- net MICROSD_CS renamed BUZZER_2
- net TEMPERATURE_SENSOR_BUS renamed T_CS
- net WOOD_AC_PRESENT renamed LED_R
- new net DISPLAY_CS: U1.30 (GPIO17)
- no-connect marks 17 -> 16
Other:
- note added: "GPIO kiosztás: GPIO18 SPI_SCK (Display SCK, T_CLK) GPIO19 SPI_MISO (Display SDO, T_DO) GPIO23 SPI_MOSI (Display SDI, T_DIN) GPIO17 DISPLAY_CS GPIO16 DISPLAY_DC GPIO04 DISPLAY_RESET GPIO32 DISPLAY_LED GPIO27 T_CS GPIO34 T_IRQ GPIO21 I2C_SDA GPIO22 I2C_SCL GPIO35 PHOTORESISTOR GPIO33 LED_R GPIO25 LED_G GPIO26 LED_B GPIO13 BUZZER_2 GPIO14 BUZZER_1"
- note removed: "GPIO kiosztás: GPIO23 SPI_MOSI GPIO19 SPI_MISO GPIO18 SPI_SCK GPIO22 I2C_SCL GPIO21 I2C_SDA GPIO27 TEMPERATURE_SENSOR_BUS (5× DS18B20) GPIO26 BOILER_ROOM_TEMPERATURE (DHT11) GPIO17 DISPLAY1_DC + DISPLAY2_DC GPIO16 DISPLAY1_RESET + DISPLAY2_RESET GPIO5 DISPLAY1_CS GPIO4 DISPLAY2_CS GPIO14 CHIMNEY_TEMPERATURE_CS (MAX6675) GPIO25 BUZZER GPIO32 GAS_AC_PRESENT GPIO33 WOOD_AC_PRESENT GPIO13 MICROSD_CS"
Changed lines of the file:
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@@
 		(comment 3 "ESP32 DevKit")
 	)
-	(text "GPIO kiosztás:\nGPIO23 SPI_MOSI\nGPIO19 SPI_MISO\nGPIO18 SPI_SCK\n\nGPIO22 I2C_SCL\nGPIO21 I2C_SDA\n\nGPIO27 TEMPERATURE_SENSOR_BUS (5× DS18B20)\n\nGPIO26 BOILER_ROOM_TEMPERATURE (DHT11)\n\nGPIO17 DISPLAY1_DC + DISPLAY2_DC\nGPIO16 DISPLAY1_RESET + DISPLAY2_RESET\nGPIO5  DISPLAY1_CS\nGPIO4  DISPLAY2_CS\n\nGPIO14 CHIMNEY_TEMPERATURE_CS (MAX6675)\n\nGPIO25 BUZZER\n\nGPIO32 GAS_AC_PRESENT\nGPIO33 WOOD_AC_PRESENT\n\nGPIO13 MICROSD_CS"
+	(text "GPIO kiosztás:\nGPIO18 SPI_SCK (Display SCK, T_CLK)\nGPIO19 SPI_MISO (Display SDO, T_DO)\nGPIO23 SPI_MOSI (Display SDI, T_DIN)\n\nGPIO17 DISPLAY_CS\nGPIO16 DISPLAY_DC\nGPIO04 DISPLAY_RESET\nGPIO32 DISPLAY_LED\n\nGPIO27 T_CS\nGPIO34 T_IRQ\n\nGPIO21 I2C_SDA\nGPIO22 I2C_SCL\n\nGPIO35 PHOTORESISTOR\n\nGPIO33 LED_R\nGPIO25 LED_G\nGPIO26 LED_B\n\nGPIO13 BUZZER_2\nGPIO14 BUZZER_1"
 		(exclude_from_sim no)
-		(at 21.59 48.006 0)
-		(effects
-			(font
-				(size 1.27 1.27)
-			)
-			(justify left)
-		)
+		(at 69.342 62.484 0)
+		(effects
+			(font
+				(size 1.27 1.27)
+			)
+			(justify left)
+		)
+	)
+	(junction
+		(at 121.92 110.49)
+		(diameter 0)
+		(color 0 0 0 0)
 	)
 	(junction
@@
 		(color 0 0 0 1)
 	)
-	(junction
-		(at 121.92 110.49)
-		(diameter 0)
-		(color 0 0 0 1)
-	)
 	(no_connect
 		(at 121.92 68.58)
@@
 	)
 	(no_connect
+		(at 121.92 121.92)
+	)
+	(no_connect
+		(at 121.92 72.39)
+	)
+	(no_connect
 		(at 121.92 106.68)
 	)
 	(no_connect
-		(at 121.92 121.92)
-	)
-	(no_connect
-		(at 121.92 72.39)
-	)
-	(no_connect
 		(at 121.92 64.77)
 	)
 	(no_connect
-		(at 121.92 80.01)
-	)
-	(no_connect
 		(at 177.8 114.3)
 	)
@@
 	)
 	(no_connect
-		(at 121.92 76.2)
+		(at 177.8 95.25)
 	)
 	(no_connect
@@
 	(wire
 		(pts
-			(xy 113.03 129.54) (xy 121.92 129.54)
+			(xy 115.57 129.54) (xy 121.92 129.54)
 		)
 		(stroke
@@
 	(wire
 		(pts
-			(xy 111.76 110.49) (xy 121.92 110.49)
+			(xy 114.3 110.49) (xy 121.92 110.49)
 		)
 		(stroke
@@
 	(wire
 		(pts
+			(xy 114.3 60.96) (xy 121.92 60.96)
+		)
+		(stroke
+			(width 0)
+			(type default)
+		)
+	)
+	(wire
+		(pts
 			(xy 121.92 110.49) (xy 158.75 110.49)
 		)
@@
 	(hierarchical_label "DISPLAY_RESET"
 		(shape output)
-		(at 177.8 102.87 0)
-		(effects
-			(font
-				(size 1.27 1.27)
-			)
-			(justify left)
-		)
-	)
-	(hierarchical_label "CHIMNEY_TEMPERATURE_CS"
+		(at 177.8 106.68 0)
+		(effects
+			(font
+				(size 1.27 1.27)
+			)
+			(justify left)
+		)
+	)
+	(hierarchical_label "PHOTORESISTOR"
 		(shape input)
-		(at 121.92 102.87 180)
+		(at 121.92 80.01 180)
 		(effects
 			(font
@@
 		)
 	)
-	(hierarchical_label "DISPLAY1_CS"
-		(shape output)
-		(at 177.8 95.25 0)
-		(effects
-			(font
-				(size 1.27 1.27)
-			)
-			(justify left)
-		)
-	)
-	(hierarchical_label "DISPLAY2_CS"
-		(shape output)
-		(at 177.8 106.68 0)
-		(effects
-			(font
-				(size 1.27 1.27)
-			)
-			(justify left)
+	(hierarchical_label "BUZZER_2"
+		(shape output)
+		(at 121.92 114.3 180)
+		(effects
+			(font
+				(size 1.27 1.27)
+			)
+			(justify right)
+		)
+	)
+	(hierarchical_label "DISPLAY_CS"
+		(shape output)
+		(at 177.8 99.06 0)
+		(effects
+			(font
+				(size 1.27 1.27)
+			)
+			(justify left)
+		)
+	)
+	(hierarchical_label "T_CS"
+		(shape output)
+		(at 121.92 99.06 180)
+		(effects
+			(font
+				(size 1.27 1.27)
+			)
+			(justify right)
 		)
 	)
@@
 		)
 	)
-	(hierarchical_label "BUZZER"
+	(hierarchical_label "BUZZER_1"
+		(shape output)
+		(at 121.92 102.87 180)
+		(effects
+			(font
+				(size 1.27 1.27)
+			)
+			(justify right)
+		)
+	)
+	(hierarchical_label "LED_R"
+		(shape output)
+		(at 121.92 87.63 180)
+		(effects
+			(font
+				(size 1.27 1.27)
+			)
+			(justify right)
+		)
+	)
+	(hierarchical_label "PWR_3V3_OUT"
+		(shape output)
+		(at 114.3 60.96 180)
+		(effects
+			(font
+				(size 1.27 1.27)
+			)
+			(justify right)
+		)
+	)
+	(hierarchical_label "LED_G"
 		(shape output)
 		(at 121.92 91.44 180)
-		(effects
-			(font
-				(size 1.27 1.27)
-			)
-			(justify right)
-		)
-	)
-	(hierarchical_label "PWR_3V3_OUT"
-		(shape output)
-		(at 121.92 60.96 180)
-		(effects
-			(font
-				(size 1.27 1.27)
-			)
-			(justify right)
-		)
-	)
-	(hierarchical_label "TEMPERATURE_SENSOR_BUS"
-		(shape input)
-		(at 121.92 99.06 180)
 		(effects
 			(font
@@
 	(hierarchical_label "PWR_5V_IN"
 		(shape input)
-		(at 113.03 129.54 180)
-		(effects
-			(font
-				(size 1.27 1.27)
-			)
-			(justify right)
-		)
-	)
-	(hierarchical_label "BOILER_ROOM_TEMPERATURE"
-		(shape input)
-		(at 121.92 95.25 180)
+		(at 115.57 129.54 180)
+		(effects
+			(font
+				(size 1.27 1.27)
+			)
+			(justify right)
+		)
+	)
+	(hierarchical_label "T_IRQ"
+		(shape output)
+		(at 121.92 76.2 180)
 		(effects
 			(font
@@
 	(hierarchical_label "PWR_GND"
 		(shape input)
-		(at 111.76 110.49 180)
+		(at 114.3 110.49 180)
 		(effects
 			(font
@@
 	(hierarchical_label "DISPLAY_DC"
 		(shape output)
-		(at 177.8 99.06 0)
-		(effects
-			(font
-				(size 1.27 1.27)
-			)
-			(justify left)
+		(at 177.8 102.87 0)
+		(effects
+			(font
+				(size 1.27 1.27)
+			)
+			(justify left)
+		)
+	)
+	(hierarchical_label "LED_B"
+		(shape output)
+		(at 121.92 95.25 180)
+		(effects
+			(font
+				(size 1.27 1.27)
+			)
+			(justify right)
 		)
 	)
@@
 		)
 	)
-	(hierarchical_label "MICROSD_CS"
-		(shape output)
-		(at 121.92 114.3 180)
-		(effects
-			(font
-				(size 1.27 1.27)
-			)
-			(justify right)
-		)
-	)
-	(hierarchical_label "WOOD_AC_PRESENT"
-		(shape input)
-		(at 121.92 87.63 180)
-		(effects
-			(font
-				(size 1.27 1.27)
-			)
-			(justify right)
-		)
-	)
-	(hierarchical_label "GAS_AC_PRESENT"
-		(shape input)
+	(hierarchical_label "DISPLAY_LED"
+		(shape output)
 		(at 121.92 83.82 180)
 		(effects
@@
 			)
 		)
-		(property "Footprint" "HMS_Footprints:ESP32_DEVKITC_32UE"
+		(property "Footprint" "HMS:ESP32_DEVKITC_32UE"
 			(at 134.62 57.15 0)
 			(hide yes)
@@
 		)
 		(instances
-			(project "HMS_Master"
+			(project "HMS_Display"
 				(path "/cab65a7d-0a7e-481c-9f85-25eca3c1fa1e/856812e0-5d79-4de2-b8e2-1ff3e02bf923"
 					(reference "U1")
