File: KiCad/HMS_Display/Sheets/02_Power_Supply.kicad_sch (KiCad schematic)
At the start: 4 parts, among them U26 USB_Micro-B_Socket

Commit message: HMS_Diaply Kicad schematics and PCB
Parts:
- U2: renamed from U26; value USB_Micro-B_Socket -> USB-C_POWER_CONNECTOR
Changed lines of the file:
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@@
 	)
 	(rectangle
-		(start 119.38 74.93)
+		(start 115.57 74.93)
 		(end 203.2 123.19)
 		(stroke
@@
 		(at 181.61 92.71)
 		(diameter 0)
-		(color 0 0 0 0)
+		(color 255 0 0 1)
 	)
 	(junction
@@
 		(at 182.88 118.11)
 		(diameter 0)
-		(color 0 0 0 0)
+		(color 0 0 0 1)
 	)
 	(junction
@@
 		)
 		(instances
-			(project "HMS_Master"
+			(project "HMS_Display"
 				(path "/cab65a7d-0a7e-481c-9f85-25eca3c1fa1e/cc839e62-2bf5-48e4-87b9-622d38cad52b"
 					(reference "#FLG02")
@@
 		)
 		(instances
-			(project "HMS_Master"
+			(project "HMS_Display"
 				(path "/cab65a7d-0a7e-481c-9f85-25eca3c1fa1e/cc839e62-2bf5-48e4-87b9-622d38cad52b"
 					(reference "C1470µF/10V1")
@@
 		)
 		(instances
-			(project "HMS_Master"
+			(project "HMS_Display"
 				(path "/cab65a7d-0a7e-481c-9f85-25eca3c1fa1e/cc839e62-2bf5-48e4-87b9-622d38cad52b"
 					(reference "#FLG01")
@@
 		)
 		(instances
-			(project "HMS_Master"
+			(project "HMS_Display"
 				(path "/cab65a7d-0a7e-481c-9f85-25eca3c1fa1e/cc839e62-2bf5-48e4-87b9-622d38cad52b"
 					(reference "C2100nF/50V1")
@@
 		(dnp no)
 		(fields_autoplaced yes)
-		(property "Reference" "U26"
+		(property "Reference" "U2"
 			(at 129.54 85.09 90)
 			(show_name no)
@@
 			)
 		)
-		(property "Value" "USB_Micro-B_Socket"
+		(property "Value" "USB-C_POWER_CONNECTOR"
 			(at 129.54 87.63 90)
 			(show_name no)
@@
 		)
 		(instances
-			(project "HMS_Master"
+			(project "HMS_Display"
 				(path "/cab65a7d-0a7e-481c-9f85-25eca3c1fa1e/cc839e62-2bf5-48e4-87b9-622d38cad52b"
-					(reference "U26")
+					(reference "U2")
 					(unit 1)
 				)
@@
 		(in_pos_files yes)
 		(dnp no)
-		(fields_autoplaced yes)
 		(property "Reference" "F1"
-			(at 143.5099 90.17 0)
+			(at 146.05 94.742 90)
 			(show_name no)
 			(do_not_autoplace no)
@@
 		)
 		(property "Value" "T1A Fuse"
-			(at 146.0499 90.17 0)
+			(at 149.098 90.932 90)
 			(show_name no)
 			(do_not_autoplace no)
@@
 		)
 		(instances
-			(project "HMS_Master"
+			(project "HMS_Display"
 				(path "/cab65a7d-0a7e-481c-9f85-25eca3c1fa1e/cc839e62-2bf5-48e4-87b9-622d38cad52b"
 					(reference "F1")
