File: KiCad/HMS_Display/Sheets/05_RTC.kicad_sch (KiCad schematic)
At the start: 1 part, among them U9 DS3231+AT24C32

Commit message: HMS_Diaply Kicad schematics and PCB
Parts:
- renumbered U9 to U8
Changed lines of the file:
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@@
 		(in_pos_files yes)
 		(dnp no)
-		(property "Reference" "U9"
+		(property "Reference" "U8"
 			(at 150.368 101.854 0)
 			(show_name no)
@@
 		)
 		(instances
-			(project "HMS_Master"
+			(project "HMS_Display"
 				(path "/cab65a7d-0a7e-481c-9f85-25eca3c1fa1e/9bf8bcb7-7800-41c3-a2be-8bb28cb524d4"
-					(reference "U9")
+					(reference "U8")
 					(unit 1)
 				)
